File: esp03_ledbar.sch (KiCad schematic (older format))
At the start: 14 parts, among them J1 CONN_01X03, J2 CONN_02X03, Q1 2N7002, U1 MP1584_MODULE, U2 ESP8266-ESP-03, U3 AP1117-33

Commit message: Migrate to new eeschema format
Parts:
- C1, C2: symbol C -> device:C
- D1: symbol LED -> device:LED
- J1: symbol CONN_01X03 -> esp03_ledbar-rescue:CONN_01X03-RESCUE-esp03_ledbar
- J2: symbol CONN_02X03 -> esp03_ledbar-rescue:CONN_02X03-RESCUE-esp03_ledbar
- Q1: symbol 2N7002 -> esp03_ledbar-rescue:2N7002-RESCUE-esp03_ledbar
- R1, R2, R3, R5: symbol R -> device:R
- R4: value 10k -> 2k; symbol R -> device:R
- U1: symbol MP1584_MODULE -> mp1584_module:MP1584_MODULE
- U2: symbol ESP8266-ESP-03 -> esp8266-esp-03:ESP8266-ESP-03
- U3: symbol AP1117-33 -> regul:AP1117-33
Connections:
- wire segments 57 -> 69
Changed lines of the file:
@@
-EESchema Schematic File Version 2
-LIBS:74xgxx
-LIBS:74xx
-LIBS:ac-dc
-LIBS:actel
-LIBS:adc-dac
-LIBS:allegro
-LIBS:Altera
-LIBS:analog_devices
-LIBS:analog_switches
-LIBS:atmel
-LIBS:audio
-LIBS:battery_management
-LIBS:bbd
-LIBS:bosch
-LIBS:brooktre
-LIBS:cmos4000
-LIBS:cmos_ieee
-LIBS:conn
-LIBS:contrib
-LIBS:cypress
-LIBS:dc-dc
-LIBS:device
-LIBS:digital-audio
-LIBS:diode
-LIBS:display
-LIBS:dsp
-LIBS:elec-unifil
-LIBS:ESD_Protection
-LIBS:ftdi
-LIBS:gennum
-LIBS:graphic
-LIBS:hc11
-LIBS:infineon
-LIBS:intel
-LIBS:interface
-LIBS:intersil
-LIBS:ir
-LIBS:Lattice
-LIBS:leds
-LIBS:LEM
-LIBS:linear
-LIBS:logo
-LIBS:maxim
-LIBS:mechanical
-LIBS:memory
-LIBS:microchip
-LIBS:microchip_dspic33dsc
-LIBS:microchip_pic10mcu
-LIBS:microchip_pic12mcu
-LIBS:microchip_pic16mcu
-LIBS:microchip_pic18mcu
-LIBS:microchip_pic24mcu
-LIBS:microchip_pic32mcu
-LIBS:microcontrollers
-LIBS:modules
-LIBS:motor_drivers
-LIBS:motorola
-LIBS:motors
-LIBS:msp430
-LIBS:nordicsemi
-LIBS:nxp
-LIBS:nxp_armmcu
-LIBS:onsemi
-LIBS:opto
-LIBS:Oscillators
-LIBS:philips
-LIBS:power
-LIBS:powerint
-LIBS:Power_Management
-LIBS:pspice
-LIBS:references
-LIBS:regul
-LIBS:relays
-LIBS:rfcom
-LIBS:RFSolutions
-LIBS:sensors
-LIBS:silabs
-LIBS:siliconi
-LIBS:stm8
-LIBS:stm32
-LIBS:supertex
-LIBS:switches
-LIBS:texas
-LIBS:transf
-LIBS:transistors
-LIBS:triac_thyristor
-LIBS:ttl_ieee
-LIBS:valves
-LIBS:video
-LIBS:wiznet
-LIBS:Worldsemi
-LIBS:Xicor
-LIBS:xilinx
-LIBS:zetex
-LIBS:Zilog
-LIBS:esp8266-esp-03
-LIBS:mp1584_module
+EESchema Schematic File Version 4
 LIBS:esp03_ledbar-cache
 EELAYER 26 0
@@
 $EndDescr
 $Comp
-L ESP8266-ESP-03 U2
+L esp8266-esp-03:ESP8266-ESP-03 U2
 U 1 1 59219788
 P 6900 2375
@@
 $EndComp
 $Comp
-L GND #PWR01
+L power:GND #PWR01
 U 1 1 59219872
 P 5900 1925
@@
 $EndComp
 $Comp
-L VCC #PWR02
+L power:VCC #PWR02
 U 1 1 592198BC
 P 5900 1700
@@
 $EndComp
 $Comp
-L VCC #PWR03
+L power:VCC #PWR03
 U 1 1 592198F0
 P 6125 1975
@@
 $EndComp
 $Comp
-L GND #PWR04
+L power:GND #PWR04
 U 1 1 59219946
 P 7950 1925
@@
 $EndComp
 $Comp
-L R R1
+L device:R R1
 U 1 1 59219996
 P 7900 1425
@@
 $EndComp
 $Comp
-L VCC #PWR05
+L power:VCC #PWR05
 U 1 1 59219A18
 P 7900 1125
@@
 $EndComp
 $Comp
-L C C1
+L device:C C1
 U 1 1 59219C0A
 P 3450 1550
@@
 $EndComp
 $Comp
-L C C2
+L device:C C2
 U 1 1 59219C48
 P 4550 1550
@@
 $EndComp
 $Comp
-L GND #PWR06
+L power:GND #PWR06
 U 1 1 59219D10
 P 3950 2075
@@
 $EndComp
 $Comp
-L VCC #PWR07
+L power:VCC #PWR07
 U 1 1 59219DCE
 P 4725 1250
@@
 $EndComp
 $Comp
-L +5V #PWR08
+L power:+5V #PWR08
 U 1 1 59219E44
 P 3075 1250
@@
 RX
 $Comp
-L CONN_01X03 J1
+L esp03_ledbar-rescue:CONN_01X03-RESCUE-esp03_ledbar J1
 U 1 1 5921A27B
 P 4600 5000
@@
 $EndComp
 $Comp
-L +5V #PWR09
+L power:+5V #PWR09
 U 1 1 5921A40A
 P 5175 4800
@@
 $EndComp
 $Comp
-L GND #PWR010
+L power:GND #PWR010
 U 1 1 5921A453
 P 5175 5200
@@
 RX
 $Comp
-L +5V #PWR011
+L power:+5V #PWR011
 U 1 1 5921B1F2
 P 2650 1500
@@
 $EndComp
 $Comp
-L GND #PWR012
+L power:GND #PWR012
 U 1 1 5921B2E0
 P 2650 2075
@@
 NoConn ~ 7475 2275
 $Comp
-L AP1117-33 U3
+L regul:AP1117-33 U3
 U 1 1 595FB7AE
 P 3950 1400
@@
 $EndComp
 $Comp
-L MP1584_MODULE U1
+L mp1584_module:MP1584_MODULE U1
 U 1 1 595FBD4A
 P 1750 1750
@@
 $EndComp
 $Comp
-L 2N7002 Q1
+L esp03_ledbar-rescue:2N7002-RESCUE-esp03_ledbar Q1
 U 1 1 595FC729
 P 2850 5025
@@
 $EndComp
 $Comp
-L R R2
+L device:R R2
 U 1 1 595FC97D
 P 2350 4925
@@
 $EndComp
 $Comp
-L R R4
+L device:R R4
 U 1 1 595FCA24
 P 3350 4925
 F 0 "R4" H 3420 4971 50  0000 L CNN
-F 1 "10k" H 3420 4880 50  0000 L CNN
+F 1 "2k" H 3420 4880 50  0000 L CNN
 F 2 "Resistors_SMD:R_0603_HandSoldering" V 3280 4925 50  0001 C CNN
 F 3 "" H 3350 4925 50  0001 C CNN
@@
 $EndComp
 $Comp
-L VCC #PWR013
+L power:VCC #PWR013
 U 1 1 595FCE83
 P 2350 4550
@@
 $EndComp
 $Comp
-L +5V #PWR014
+L power:+5V #PWR014
 U 1 1 595FCED3
 P 3350 4525
@@
 LEVEL SHIFTER
 $Comp
-L R R3
+L device:R R3
 U 1 1 595FD05C
 P 2850 5500
@@
 	7475 1975 7900 1975
 Wire Wire Line
-	7475 1775 8225 1775
+	7475 1775 7900 1775
 Wire Wire Line
 	7900 1775 7900 1575
@@
 	7900 1275 7900 1125
 Wire Wire Line
-	3075 1400 3650 1400
+	3075 1400 3450 1400
 Connection ~ 3450 1400
 Wire Wire Line
 	3450 1700 3450 1850
 Wire Wire Line
-	3450 1850 4550 1850
-Wire Wire Line
-	3950 1700 3950 2075
+	3450 1850 3950 1850
+Wire Wire Line
+	3950 1700 3950 1850
 Connection ~ 3950 1850
 Wire Wire Line
 	4550 1850 4550 1700
 Wire Wire Line
-	4250 1400 4725 1400
+	4250 1400 4550 1400
 Wire Wire Line
 	4725 1400 4725 1250
@@
 	2500 1600 2500 1500
 Wire Wire Line
-	2350 1500 2650 1500
+	2350 1500 2500 1500
 Connection ~ 2500 1500
 Wire Wire Line
@@
 	2500 1900 2500 2000
 Wire Wire Line
-	2350 2000 2650 2000
+	2350 2000 2500 2000
 Wire Wire Line
 	2650 2000 2650 2075
@@
 	7900 1925 7950 1925
 Wire Wire Line
-	1925 5125 2650 5125
-Wire Wire Line
-	2350 5075 2350 5500
+	1925 5125 2350 5125
+Wire Wire Line
+	2350 5075 2350 5125
 Connection ~ 2350 5125
 Wire Wire Line
-	3050 5125 3950 5125
-Wire Wire Line
-	3350 5075 3350 5500
+	3050 5125 3350 5125
+Wire Wire Line
+	3350 5075 3350 5125
 Connection ~ 3350 5125
 Wire Wire Line
@@
 	2850 4675 2350 4675
 Wire Wire Line
-	2350 4550 2350 4775
+	2350 4550 2350 4675
 Connection ~ 2350 4675
 Wire Wire Line
@@
 	1000 2600 1000 700
 $Comp
-L CONN_02X03 J2
+L esp03_ledbar-rescue:CONN_02X03-RESCUE-esp03_ledbar J2
 U 1 1 59600EF5
 P 9300 1750
@@
 	9850 1850 9850 1900
 $Comp
-L GND #PWR015
+L power:GND #PWR015
 U 1 1 596013EF
 P 9850 1900
@@
 $EndComp
 $Comp
-L VCC #PWR016
+L power:VCC #PWR016
 U 1 1 59601474
 P 9850 1650
@@
 $EndComp
 $Comp
-L LED D1
+L device:LED D1
 U 1 1 5960186A
 P 9350 2550
@@
 $EndComp
 $Comp
-L R R5
+L device:R R5
 U 1 1 596018FD
 P 8950 2550
@@
 $EndComp
 $Comp
-L GND #PWR017
+L power:GND #PWR017
 U 1 1 5960194A
 P 8700 2650
@@
 $EndComp
 $Comp
-L VCC #PWR018
+L power:VCC #PWR018
 U 1 1 59601971
 P 9700 2450
@@
 	8700 2550 8700 2650
 NoConn ~ 9550 1650
+Wire Wire Line
+	3450 1400 3650 1400
+Wire Wire Line
+	3950 1850 4550 1850
+Wire Wire Line
+	3950 1850 3950 2075
+Wire Wire Line
+	4550 1400 4725 1400
+Wire Wire Line
+	7900 1775 8225 1775
+Wire Wire Line
+	2500 1500 2650 1500
+Wire Wire Line
+	2500 2000 2650 2000
+Wire Wire Line
+	2350 5125 2650 5125
+Wire Wire Line
+	2350 5125 2350 5500
+Wire Wire Line
+	3350 5125 3950 5125
+Wire Wire Line
+	3350 5125 3350 5500
+Wire Wire Line
+	2350 4675 2350 4775
 $EndSCHEMATC
